Commit message: feat: complete aquatic simulation with buoy arena, APF navigation and RViz waypoint tracking
- Added closed_aquatic_arena.world with 42 marine buoys (slalom and hazard markers)
- Implemented boat_waypoint_nav.py with Artificial Potential Fields (APF) and 2D Nav Goal
- Added RViz config with real-time 3D force vector arrows (Attraction, Repulsion, Total)
- Fixed IMU and propeller joint TF publishers for migbot1
- Added boat_aquatic_arena.launch with full simulation and autonomous navigation
- Updated README with quick start and project documentation

File: robots/migbot_description/urdf/migbot1.urdf.xacro (robot description, xacro)
@@ -209,11 +209,8 @@
     </sensor>
   </link>
-  <joint name="imu_joint" type="revolute">
+  <joint name="imu_joint" type="fixed">
     <parent link="base_link"/>
     <child link="imu_link"/>
     <origin rpy="0 0 0" xyz="-0.01 0.002 0.082"/>
-    <axis xyz="1 0 0"/>
-    <limit effort="0.0" lower="0" upper="0" velocity="0"/>
-    <dynamics damping="0.7" friction="0" spring_reference="0" spring_stiffness="0"/>
   </joint>
   <gazebo reference="imu_link">

File: robots/migbot_description/urdf/migbot1_ardupilot.urdf.xacro (robot description, xacro)
@@ -200,11 +200,8 @@
     </sensor>
   </link>
-  <joint name="imu_joint" type="revolute">
+  <joint name="imu_joint" type="fixed">
     <parent link="base_link"/>
     <child link="imu_link"/>
     <origin rpy="0 0 0" xyz="-0.01 0.002 0.082"/>
-    <axis xyz="1 0 0"/>
-    <limit effort="0.0" lower="0" upper="0" velocity="0"/>
-    <dynamics damping="0.7" friction="0" spring_reference="0" spring_stiffness="0"/>
   </joint>
   <gazebo reference="imu_link">

File: robots/migbot_description/urdf/migbot1_ros.urdf.xacro (robot description, xacro)
@@ -209,11 +209,8 @@
     </sensor>
   </link>
-  <joint name="imu_joint" type="revolute">
+  <joint name="imu_joint" type="fixed">
     <parent link="base_link"/>
     <child link="imu_link"/>
     <origin rpy="0 0 0" xyz="-0.01 0.002 0.082"/>
-    <axis xyz="1 0 0"/>
-    <limit effort="0.0" lower="0" upper="0" velocity="0"/>
-    <dynamics damping="0.7" friction="0" spring_reference="0" spring_stiffness="0"/>
   </joint>
   <gazebo reference="imu_link">

File: robots/migbot_gazebo/urdf/macros_migbot.xacro (robot description, xacro)
@@ -1,10 +1,9 @@
 <?xml version="1.0"?>
 <!-- Includes all macros in this package so they don't need to be included individualy -->
-<robot xmlns:xacro="http://ros.org/wiki/xacro"
-       name="migbot1">
-  <!-- Include dynamics macros -->
+<robot xmlns:xacro="http://ros.org/wiki/xacro" name="migbot1">
   <!-- Include sensor macros -->
   <xacro:include filename="$(find migbot_gazebo)/urdf/components/Livox_Mid70_mount.xacro" />
   <xacro:include filename="$(find migbot_gazebo)/urdf/components/ping360_mount.xacro" />
   <xacro:include filename="$(find migbot_gazebo)/urdf/components/realsensed435_mount.xacro" />
+  <xacro:include filename="$(find migbot_gazebo)/urdf/components/planar_lidar_mount.xacro" />
 </robot>

File: robots/migbot_gazebo/urdf/migbot_gazebo.urdf.xacro (robot description, xacro)
@@ -1,4 +1,6 @@
 <?xml version="1.0"?>
 <robot xmlns:xacro="http://ros.org/wiki/xacro" name="migbot1">
+  <xacro:arg name="planar_move_enabled" default="true" />
+  <xacro:arg name="planar_lidar_enabled" default="false" />
   <xacro:arg name="livox_enabled" default="false" />
   <xacro:arg name="ping360_enabled" default="false" />
@@ -29,3 +31,20 @@
 	    prefix ="realsense"/>
     </xacro:if>
+    <!-- Add 2D Planar LIDAR -->
+    <xacro:if value="$(arg planar_lidar_enabled)">
+        <xacro:planar_lidar_mount name="laser" topic="/scan" />
+    </xacro:if>
+    <!-- Planar Movement Plugin (for reliable non-holonomic boat control via /cmd_vel) -->
+    <xacro:if value="$(arg planar_move_enabled)">
+      <gazebo>
+        <plugin name="planar_move" filename="libgazebo_ros_planar_move.so">
+          <commandTopic>/cmd_vel</commandTopic>
+          <odometryTopic>/odom</odometryTopic>
+          <odometryFrame>odom</odometryFrame>
+          <odometryRate>30.0</odometryRate>
+          <robotBaseFrame>base_link</robotBaseFrame>
+          <enableYAxis>false</enableYAxis>
+        </plugin>
+      </gazebo>
+    </xacro:if>
 </robot>
